Commit message: Agregando archivos de código fuente y URDF completos

File: src/x3plus_description/urdf/x3plus_chassis.xacro (robot description, xacro)
@@ -60,5 +60,5 @@
             <mu1>100.0</mu1>
             <mu2>100.0</mu2>
-            <kp>10000000.0</kp>
+            <kp>100000.0</kp>
             <kd>1.0</kd>
             <minDepth>0.005</minDepth>

File: src/x3plus_description/urdf/x3plus_control.xacro (robot description, xacro)
@@ -36,12 +36,7 @@
                 <state_interface name="position"/>
                 <state_interface name="velocity"/>
-                </joint>
+            </joint>
         </xacro:macro>
-        <xacro:gripper_control joint_name="grip_joint"/>
-        <xacro:gripper_control joint_name="rfinger_joint_01"/>
-        <xacro:gripper_control joint_name="rfinger_joint_02"/>
-        <xacro:gripper_control joint_name="lfinger_grip_joint_01"/>
-        <xacro:gripper_control joint_name="lfinger_grip_joint_02"/>
-        <xacro:gripper_control joint_name="lfinger_grip_joint_03"/>
+        <xacro:gripper_control joint_name="joint6_gripper"/>
     </ros2_control>
     <gazebo>
