Commit message: Respaldo estable: física corregida, brazo alineado y sensores con masa

File: src/x3plus_description/urdf/x3plus_accessories.xacro (robot description, xacro)
@@ -3,42 +3,6 @@
     <joint name="omni_to_dofbot_joint" type="fixed">
         <origin xyz="0.1025 0 0.031" rpy="0 0 -1.57" />
-        <parent link="base_footprint" />
+        <parent link="base_link" />
         <child link="arm_pedestal_link" />
     </joint>
-    <link name="mastil_link">
-        <visual>
-            <origin xyz="0 0 0.1775" rpy="0 0 0"/>
-            <geometry><box size="0.02 0.04 0.355"/></geometry>
-            <material name="grey"><color rgba="0.5 0.5 0.5 1.0"/></material>
-        </visual>
-        <collision>
-            <origin rpy="0 0 0" xyz="0 0 0.1775"/>
-            <geometry><box size="0.02 0.04 0.355"/></geometry>
-        </collision>
-    </link>
-    <joint name="base_to_mastil_joint" type="fixed">
-        <origin xyz="-0.035 0 0.0615" rpy="0 0 0"/>
-        <parent link="base_footprint"/>
-        <child link="mastil_link"/>
-    </joint>
-    <link name="display_link">
-        <visual>
-            <origin rpy="0 0 0" xyz="0 0 0"/>
-            <geometry>
-                <mesh filename="file://$(find x3plus_description)/meshes/display_omni_dofbot.stl"/>
-            </geometry>
-            <material name="blue"><color rgba="0 0.7 0 1"/></material>
-        </visual>
-        <collision>
-            <origin rpy="0 0 0" xyz="0 0 0"/>
-            <geometry>
-                <mesh filename="file://$(find x3plus_description)/meshes/display_omni_dofbot.stl"/>
-            </geometry>
-        </collision>
-    </link>
-    <joint name="display_joint" type="fixed">
-        <parent link="mastil_link"/>
-        <child link="display_link"/>
-        <origin rpy="0 0 0" xyz="-0.07 0.0 0.265"/>
-    </joint>
 </robot>

File: src/x3plus_description/urdf/x3plus_chassis.xacro (robot description, xacro)
@@ -36,11 +36,18 @@
     </link>
     <joint name="base_to_tower" type="fixed"><parent link="base_link"/><child link="sensor_tower_link"/><origin xyz="-0.10 0 0.05" rpy="0 0 0"/></joint>
-    <link name="tower_camera_link"><visual><origin xyz="0 0 0" rpy="0 0 0"/><geometry><box size="0.02 0.10 0.025"/></geometry><material name="metal_black"/></visual></link>
+    <link name="tower_camera_link">
+        <visual><origin xyz="0 0 0" rpy="0 0 0"/><geometry><box size="0.02 0.10 0.025"/></geometry><material name="metal_black"/></visual>
+        <inertial><mass value="0.05"/><inertia ixx="0.0001" ixy="0" ixz="0" iyy="0.0001" iyz="0" izz="0.0001"/></inertial>
+    </link>
     <joint name="tower_to_camera" type="fixed"><parent link="sensor_tower_link"/><child link="tower_camera_link"/><origin xyz="0.03 0 0.40" rpy="0 0 0"/></joint>
-    <link name="display_panel_link"><visual><origin xyz="0 0 0" rpy="0 0 0"/><geometry><box size="0.01 0.12 0.18"/></geometry><material name="panel_blue"/></visual></link>
+    <link name="display_panel_link">
+        <visual><origin xyz="0 0 0" rpy="0 0 0"/><geometry><box size="0.01 0.12 0.18"/></geometry><material name="panel_blue"/></visual>
+        <inertial><mass value="0.05"/><inertia ixx="0.0001" ixy="0" ixz="0" iyy="0.0001" iyz="0" izz="0.0001"/></inertial>
+    </link>
     <joint name="tower_to_display" type="fixed"><parent link="sensor_tower_link"/><child link="display_panel_link"/><origin xyz="-0.03 0 0.30" rpy="0 -0.2 0"/></joint>
     <link name="antenna_link">
         <visual><origin xyz="0 -0.02 0.06" rpy="0 0.3 0"/><geometry><cylinder radius="0.005" length="0.12"/></geometry><material name="metal_black"/></visual>
         <visual><origin xyz="0 0.02 0.06" rpy="0 0.3 0"/><geometry><cylinder radius="0.005" length="0.12"/></geometry><material name="metal_black"/></visual>
+        <inertial><mass value="0.01"/><inertia ixx="0.00001" ixy="0" ixz="0" iyy="0.00001" iyz="0" izz="0.00001"/></inertial>
     </link>
     <joint name="base_to_antenna" type="fixed"><parent link="base_link"/><child link="antenna_link"/><origin xyz="-0.13 0 0.05" rpy="0 0 0"/></joint>
@@ -48,4 +55,5 @@
         <visual><origin xyz="0 0 0.02" rpy="0 0 0"/><geometry><cylinder radius="0.05" length="0.04"/></geometry><material name="metal_black"/></visual>
         <collision><origin xyz="0 0 0.02" rpy="0 0 0"/><geometry><cylinder radius="0.05" length="0.04"/></geometry></collision>
+        <inertial><mass value="0.1"/><inertia ixx="0.0001" ixy="0" ixz="0" iyy="0.0001" iyz="0" izz="0.0001"/></inertial>
     </link>
     <joint name="base_to_lidar" type="fixed"><parent link="base_link"/><child link="lidar_link"/><origin xyz="-0.02 0 0.05" rpy="0 0 0"/></joint>
